Commit message: Put two UR10 on the same rail

File: osrf_gear/launch/vacuum_gripper/vacuum_gripper.urdf.xacro (robot description, xacro)
@@ -1,5 +1,5 @@
 <?xml version="1.0"?>
 <robot xmlns:xacro="http://www.ros.org/wiki/xacro">
-<xacro:macro name="create_vacuum_gripper" params="wrist_link *origin **grippable_model_types **drops_info">
+<xacro:macro name="create_vacuum_gripper" params="wrist_link arm_namespace *origin **grippable_model_types **drops_info">
   <link name="vacuum_gripper_link">
     <inertial>
@@ -51,5 +51,5 @@
       <suction_cup_link>vacuum_gripper_link</suction_cup_link>
       <!-- ROS -->
-      <robot_namespace>/ariac</robot_namespace>
+      <robot_namespace>${arm_namespace}</robot_namespace>
       <control_topic>gripper/control</control_topic>
       <state_topic>gripper/state</state_topic>
