Commit message: Make rail a model in world

File: osrf_gear/launch/linear_arm_actuator/linear_arm_actuator.urdf.xacro (robot description, xacro)
@@ -15,19 +15,4 @@
       <mass value="1" />
     </inertial>
-    <visual>
-      <origin xyz="0 0 0" rpy="0 0 0" />
-      <geometry>
-        <box size="${base_len} ${actuator_len} ${actuator_height}" />
-      </geometry>
-      <material name="Grey">
-        <color rgba="0.2 0.2 0.2 1.0"/>
-      </material>
-    </visual>
-    <collision>
-      <origin xyz="0 0 0" rpy="0 0 0" />
-      <geometry>
-        <box size="${base_len} ${actuator_len} ${actuator_height}" />
-      </geometry>
-    </collision>
   </link>
   <gazebo reference="linear_arm_actuator">

Commit message: Each arm can travel 60% of the rail

File: osrf_gear/launch/linear_arm_actuator/linear_arm_actuator.urdf.xacro (robot description, xacro)
@@ -2,5 +2,5 @@
 <robot xmlns:xacro="http://www.ros.org/wiki/xacro">
 <xacro:property name="base_len" value="0.2" />
-<xacro:property name="actuator_len" value="4.0" />
+<xacro:property name="actuator_len" value="2.4" />
 <xacro:property name="actuator_height" value="0.1" />
 <xacro:arg name="use_velocity_interface" default="false" />

Commit message: increase range of arms on rail
Signed-off-by: Shane Loretz <sloretz@osrfoundation.org>

File: osrf_gear/launch/linear_arm_actuator/linear_arm_actuator.urdf.xacro (robot description, xacro)
@@ -2,5 +2,5 @@
 <robot xmlns:xacro="http://www.ros.org/wiki/xacro">
 <xacro:property name="base_len" value="0.2" />
-<xacro:property name="actuator_len" value="2.4" />
+<xacro:property name="actuator_len" value="2.76" />
 <xacro:property name="actuator_height" value="0.1" />
 <xacro:arg name="use_velocity_interface" default="false" />
